File: hardware/mysz.brd (EAGLE design)
At the start: 160 x 100 mm, 17 parts, among them IC1 LM1117T(H)-3.3, U1 NUCLEO-L053R8, X2 332-18

Commit message: Add Gyro schemat
Parts:
- removed U$2: DISPLAY-NOKIA-3310, diy-modules:DISPLAY-NOKIA-3310
- removed X2: 332-18, con-garry:332-18
- added GYRO: (no value), pinhead:1X10
- added PCD8544: (no value), pinhead:1X07/90
- added R3, R4: 22k, rcl:0207/10
Connections:
- removed net GND.1: U$2.J1.2
- removed net GND.2: U$2.J2.2
- removed net VCC.1: U$2.J1.1
- removed net VCC.2: U$2.J2.1
- new net GYRO_CS: GYRO.3
- new net GYRO_DEN: GYRO.1
- new net GYRO_INT1: GYRO.2
- new net GYRO_SCL: GYRO.6, R3.1
- new net GYRO_SDA: GYRO.7, R4.1
- new net LCD_CE: PCD8544.2
- new net LCD_DC: PCD8544.3
- new net LCD_RST: PCD8544.1
- new net N$4: GYRO.10, GYRO.4
- net +3V3: now also R3.2, R4.2
Changed lines of the file:
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@@
 <layer number="48" name="Document" color="7" fill="1" visible="yes" active="yes"/>
 <layer number="49" name="Reference" color="7" fill="1" visible="yes" active="yes"/>
+<layer number="50" name="dxf" color="7" fill="1" visible="no" active="yes"/>
 <layer number="51" name="tDocu" color="7" fill="1" visible="yes" active="yes"/>
 <layer number="52" name="bDocu" color="7" fill="1" visible="yes" active="yes"/>
+<layer number="56" name="wert" color="7" fill="1" visible="no" active="no"/>
 <layer number="88" name="SimResults" color="9" fill="1" visible="no" active="no"/>
 <layer number="89" name="SimProbes" color="9" fill="1" visible="no" active="no"/>
@@
 <layer number="98" name="Guide" color="6" fill="1" visible="no" active="no"/>
 <layer number="99" name="SpiceOrder" color="5" fill="1" visible="no" active="no"/>
+<layer number="100" name="Mechanical" color="7" fill="1" visible="no" active="no"/>
+<layer number="101" name="Gehäuse" color="7" fill="1" visible="no" active="no"/>
+<layer number="102" name="Mittellin" color="7" fill="1" visible="no" active="no"/>
+<layer number="151" name="HeatSink" color="14" fill="1" visible="no" active="no"/>
+<layer number="200" name="200bmp" color="1" fill="10" visible="no" active="no"/>
+<layer number="250" name="Descript" color="3" fill="1" visible="no" active="no"/>
+<layer number="251" name="SMDround" color="12" fill="11" visible="no" active="no"/>
+<layer number="254" name="OrgLBR" color="13" fill="1" visible="no" active="no"/>
 </layers>
 <board>
@@
 <attribute name="VALUE" x="-71.12" y="1.27" size="1.778" layer="27"/>
 </element>
-<element name="X2" library="con-garry" library_urn="urn:adsk.eagle:library:147" package="332-18" package3d_urn="urn:adsk.eagle:package:6813/1" value="332-18" x="-62.23" y="-16.51" smashed="yes">
-<attribute name="NAME" x="-70.85" y="-13.97" size="1.27" layer="25"/>
-<attribute name="POPULARITY" value="0" x="-62.23" y="-16.51" size="1.778" layer="27" display="off"/>
-<attribute name="VALUE" x="-64.5" y="-13.97" size="1.27" layer="27"/>
-</element>
 <element name="U$1" library="diy-modules" package="WIRELESS-BLUETOOTH-HC-05" value="WIRELESS-BLUETOOTH-HC-05" x="-81.28" y="-35.56" smashed="yes">
 <attribute name="NAME" x="-81.28" y="-15.875" size="1.27" layer="25" align="bottom-center"/>
 <attribute name="VALUE" x="-81.28" y="-55.245" size="1.27" layer="27" align="top-center"/>
-</element>
-<element name="U$2" library="diy-modules" package="DISPLAY-NOKIA-3310" value="DISPLAY-NOKIA-3310" x="-118.11" y="-30.48" smashed="yes">
-<attribute name="NAME" x="-118.11" y="-6.35" size="1.27" layer="25" align="bottom-center"/>
-<attribute name="VALUE" x="-118.11" y="-54.61" size="1.27" layer="27" align="top-center"/>
 </element>
 <element name="POWER" library="pinhead" library_urn="urn:adsk.eagle:library:325" package="1X02" package3d_urn="urn:adsk.eagle:package:22435/2" value="" x="-137.16" y="-60.96" smashed="yes">
@@
 <attribute name="VALUE" x="-153.3906" y="-180.975" size="1.27" layer="27" ratio="10"/>
 </element>
+<element name="R3" library="rcl" library_urn="urn:adsk.eagle:library:334" package="0207/10" package3d_urn="urn:adsk.eagle:package:23491/2" value="22k" x="-151.13" y="-185.42" smashed="yes">
+<attribute name="NAME" x="-154.178" y="-183.896" size="1.27" layer="25" ratio="10"/>
+<attribute name="POPULARITY" value="81" x="-151.13" y="-185.42" size="1.778" layer="27" display="off"/>
+<attribute name="SPICEPREFIX" value="R" x="-151.13" y="-185.42" size="1.778" layer="27" display="off"/>
+<attribute name="VALUE" x="-153.3906" y="-186.055" size="1.27" layer="27" ratio="10"/>
+</element>
+<element name="R4" library="rcl" library_urn="urn:adsk.eagle:library:334" package="0207/10" package3d_urn="urn:adsk.eagle:package:23491/2" value="22k" x="-151.13" y="-190.5" smashed="yes">
+<attribute name="NAME" x="-154.178" y="-188.976" size="1.27" layer="25" ratio="10"/>
+<attribute name="POPULARITY" value="81" x="-151.13" y="-190.5" size="1.778" layer="27" display="off"/>
+<attribute name="SPICEPREFIX" value="R" x="-151.13" y="-190.5" size="1.778" layer="27" display="off"/>
+<attribute name="VALUE" x="-153.3906" y="-191.135" size="1.27" layer="27" ratio="10"/>
+</element>
+<element name="GYRO" library="pinhead" library_urn="urn:adsk.eagle:library:325" package="1X10" package3d_urn="urn:adsk.eagle:package:22406/2" value="" x="-143.51" y="-195.58" smashed="yes">
+<attribute name="NAME" x="-156.2862" y="-193.7512" size="1.27" layer="25" ratio="10"/>
+<attribute name="POPULARITY" value="35" x="-143.51" y="-195.58" size="1.778" layer="27" display="off"/>
+<attribute name="VALUE" x="-156.21" y="-198.755" size="1.27" layer="27"/>
+</element>
+<element name="PCD8544" library="pinhead" library_urn="urn:adsk.eagle:library:325" package="1X07/90" package3d_urn="urn:adsk.eagle:package:22476/2" value="" x="-146.05" y="-205.74" smashed="yes">
+<attribute name="NAME" x="-155.575" y="-209.55" size="1.27" layer="25" ratio="10" rot="R90"/>
+<attribute name="POPULARITY" value="1" x="-146.05" y="-205.74" size="1.778" layer="27" display="off"/>
+<attribute name="VALUE" x="-135.255" y="-209.55" size="1.27" layer="27" rot="R90"/>
+</element>
 </elements>
 <signals>
-<signal name="VCC.2">
-<contactref element="U$2" pad="J2.1"/>
-</signal>
-<signal name="GND.2">
-<contactref element="U$2" pad="J2.2"/>
-</signal>
-<signal name="VCC.1">
-<contactref element="U$2" pad="J1.1"/>
-</signal>
-<signal name="GND.1">
-<contactref element="U$2" pad="J1.2"/>
-</signal>
 <signal name="GND">
 <contactref element="U$1" pad="4"/>
@@
 <contactref element="R1" pad="2"/>
 <contactref element="R2" pad="2"/>
+<contactref element="R3" pad="2"/>
+<contactref element="R4" pad="2"/>
 <wire x1="-133.35" y1="-73.66" x2="-123.19" y2="-87.63" width="0" layer="19" extent="1-1"/>
 <wire x1="-133.35" y1="-67.31" x2="-133.35" y2="-73.66" width="0" layer="19" extent="1-1"/>
@@
 <wire x1="-146.05" y1="-175.26" x2="-140.97" y2="-170.18" width="0" layer="19" extent="1-1"/>
 <wire x1="-146.05" y1="-180.34" x2="-146.05" y2="-175.26" width="0" layer="19" extent="1-1"/>
+<wire x1="-146.05" y1="-185.42" x2="-146.05" y2="-180.34" width="0" layer="19" extent="1-1"/>
+<wire x1="-146.05" y1="-190.5" x2="-146.05" y2="-185.42" width="0" layer="19" extent="1-1"/>
 </signal>
 <signal name="ENC_L_B">
@@
 <wire x1="-3.81" y1="28.56" x2="-151.13" y2="-170.18" width="0" layer="19" extent="1-1"/>
 </signal>
+<signal name="GYRO_SCL">
+<contactref element="R3" pad="1"/>
+<contactref element="GYRO" pad="6"/>
+<wire x1="-142.24" y1="-195.58" x2="-156.21" y2="-185.42" width="0" layer="19" extent="1-1"/>
+</signal>
+<signal name="GYRO_SDA">
+<contactref element="R4" pad="1"/>
+<contactref element="GYRO" pad="7"/>
+<wire x1="-139.7" y1="-195.58" x2="-156.21" y2="-190.5" width="0" layer="19" extent="1-1"/>
+</signal>
+<signal name="GYRO_DEN">
+<contactref element="GYRO" pad="1"/>
+</signal>
+<signal name="GYRO_CS">
+<contactref element="GYRO" pad="3"/>
+</signal>
+<signal name="N$4">
+<contactref element="GYRO" pad="10"/>
+<contactref element="GYRO" pad="4"/>
+<wire x1="-132.08" y1="-195.58" x2="-147.32" y2="-195.58" width="0" layer="19" extent="1-1"/>
+</signal>
+<signal name="GYRO_INT1">
+<contactref element="GYRO" pad="2"/>
+</signal>
+<signal name="LCD_RST">
+<contactref element="PCD8544" pad="1"/>
+</signal>
+<signal name="LCD_CE">
+<contactref element="PCD8544" pad="2"/>
+</signal>
+<signal name="LCD_DC">
+<contactref element="PCD8544" pad="3"/>
+</signal>
 </signals>

Commit message: Add driver
Parts:
- removed PCD8544: (no value), pinhead:1X07/90
- added DRIVER1, DRIVER2, LCD: (no value), pinhead:1X08
Connections:
- new net GND_UC: DRIVER1.1
- new net LCD_BL: LCD.7
- new net LCD_CLK: LCD.5
- new net LCD_DIN: LCD.4
- new net N$1: DRIVER1.3
- new net N$2: DRIVER1.4
- new net N$3: DRIVER1.5
- new net N$5: DRIVER1.6
- net +3V3: now also LCD.6
- net GND: now also DRIVER2.8, LCD.8
- net LCD_CE: now also LCD.2; no longer PCD8544.2
- net LCD_DC: now also LCD.3; no longer PCD8544.3
- net LCD_RST: now also LCD.1; no longer PCD8544.1
Changed lines of the file:
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@@
 <attribute name="VALUE" x="-156.21" y="-198.755" size="1.27" layer="27"/>
 </element>
-<element name="PCD8544" library="pinhead" library_urn="urn:adsk.eagle:library:325" package="1X07/90" package3d_urn="urn:adsk.eagle:package:22476/2" value="" x="-146.05" y="-205.74" smashed="yes">
-<attribute name="NAME" x="-155.575" y="-209.55" size="1.27" layer="25" ratio="10" rot="R90"/>
-<attribute name="POPULARITY" value="1" x="-146.05" y="-205.74" size="1.778" layer="27" display="off"/>
-<attribute name="VALUE" x="-135.255" y="-209.55" size="1.27" layer="27" rot="R90"/>
+<element name="LCD" library="pinhead" library_urn="urn:adsk.eagle:library:325" package="1X08" package3d_urn="urn:adsk.eagle:package:22409/2" value="" x="-146.05" y="-201.93" smashed="yes">
+<attribute name="NAME" x="-156.2862" y="-200.1012" size="1.27" layer="25" ratio="10"/>
+<attribute name="POPULARITY" value="67" x="-146.05" y="-201.93" size="1.778" layer="27" display="off"/>
+<attribute name="VALUE" x="-156.21" y="-205.105" size="1.27" layer="27"/>
+</element>
+<element name="DRIVER1" library="pinhead" library_urn="urn:adsk.eagle:library:325" package="1X08" package3d_urn="urn:adsk.eagle:package:22409/2" value="" x="-146.05" y="-208.28" smashed="yes">
+<attribute name="NAME" x="-156.2862" y="-206.4512" size="1.27" layer="25" ratio="10"/>
+<attribute name="POPULARITY" value="67" x="-146.05" y="-208.28" size="1.778" layer="27" display="off"/>
+<attribute name="VALUE" x="-156.21" y="-211.455" size="1.27" layer="27"/>
+</element>
+<element name="DRIVER2" library="pinhead" library_urn="urn:adsk.eagle:library:325" package="1X08" package3d_urn="urn:adsk.eagle:package:22409/2" value="" x="-146.05" y="-214.63" smashed="yes">
+<attribute name="NAME" x="-156.2862" y="-212.8012" size="1.27" layer="25" ratio="10"/>
+<attribute name="POPULARITY" value="67" x="-146.05" y="-214.63" size="1.778" layer="27" display="off"/>
+<attribute name="VALUE" x="-156.21" y="-217.805" size="1.27" layer="27"/>
 </element>
 </elements>
@@
 <contactref element="VL-M" pad="5"/>
 <contactref element="VL-R" pad="5"/>
+<contactref element="LCD" pad="8"/>
+<contactref element="DRIVER2" pad="8"/>
 <wire x1="-125.73" y1="-73.66" x2="-125.73" y2="-87.63" width="0" layer="19" extent="1-1"/>
 <wire x1="-125.73" y1="-67.31" x2="-125.73" y2="-73.66" width="0" layer="19" extent="1-1"/>
@@
 <wire x1="-143.51" y1="-156.21" x2="-153.67" y2="-140.97" width="0" layer="19" extent="1-1"/>
 <wire x1="-143.51" y1="-170.18" x2="-143.51" y2="-156.21" width="0" layer="19" extent="1-1"/>
+<wire x1="-137.16" y1="-201.93" x2="-143.51" y2="-170.18" width="0" layer="19" extent="1-1"/>
+<wire x1="-137.16" y1="-214.63" x2="-137.16" y2="-201.93" width="0" layer="19" extent="1-1"/>
 <wire x1="-80.01" y1="-52.705" x2="-125.73" y2="-67.31" width="0" layer="19" extent="1-1"/>
 </signal>
@@
 <contactref element="R3" pad="2"/>
 <contactref element="R4" pad="2"/>
+<contactref element="LCD" pad="6"/>
 <wire x1="-133.35" y1="-73.66" x2="-123.19" y2="-87.63" width="0" layer="19" extent="1-1"/>
 <wire x1="-133.35" y1="-67.31" x2="-133.35" y2="-73.66" width="0" layer="19" extent="1-1"/>
@@
 <wire x1="-146.05" y1="-185.42" x2="-146.05" y2="-180.34" width="0" layer="19" extent="1-1"/>
 <wire x1="-146.05" y1="-190.5" x2="-146.05" y2="-185.42" width="0" layer="19" extent="1-1"/>
+<wire x1="-142.24" y1="-201.93" x2="-146.05" y2="-190.5" width="0" layer="19" extent="1-1"/>
 </signal>
 <signal name="ENC_L_B">
@@
 </signal>
 <signal name="LCD_RST">
-<contactref element="PCD8544" pad="1"/>
+<contactref element="LCD" pad="1"/>
 </signal>
 <signal name="LCD_CE">
-<contactref element="PCD8544" pad="2"/>
+<contactref element="LCD" pad="2"/>
 </signal>
 <signal name="LCD_DC">
-<contactref element="PCD8544" pad="3"/>
+<contactref element="LCD" pad="3"/>
+</signal>
+<signal name="LCD_DIN">
+<contactref element="LCD" pad="4"/>
+</signal>
+<signal name="LCD_CLK">
+<contactref element="LCD" pad="5"/>
+</signal>
+<signal name="LCD_BL">
+<contactref element="LCD" pad="7"/>
+</signal>
+<signal name="GND_UC">
+<contactref element="DRIVER1" pad="1"/>
+</signal>
+<signal name="N$2">
+<contactref element="DRIVER1" pad="4"/>
+</signal>
+<signal name="N$3">
+<contactref element="DRIVER1" pad="5"/>
+</signal>
+<signal name="N$5">
+<contactref element="DRIVER1" pad="6"/>
+</signal>
+<signal name="N$1">
+<contactref element="DRIVER1" pad="3"/>
 </signal>
 </signals>

Commit message: conection models to stm & stm corected
Parts:
- added C5, C8: 100nF, capacitor-wima:C2.5-3
- added C6, C7: 100uF, capacitor-wima:C2.5-3
- added IC2: LM1117T(H)-3.3, lm1117_10:TO220H
- added LED1: TLLG4400, led:LED3MM
- added R5: 1k, rcl:0207/10
Connections:
- net N$1 renamed MOTOR_BIN_R
- net N$2 renamed MOTOR_BIN_L
- net N$3 renamed MOTOR_AIN_L
- net N$5 renamed MOTOR_AIN_R
- new net BT_LED: R5.1, U1.CN7_3
- new net LS: C7.1, C8.1, IC2.2, LCD.6, U1.CN6_4, U1.CN7_16
- new net M1L: DRIVER2.3, ENC-L.1
- new net M1R: DRIVER2.6, ENC-R.1
- new net M2L: DRIVER2.4, ENC-L.2
- new net M2R: DRIVER2.5, ENC-R.2
- new net N$1: LED1.K
- new net N$2: U1.CN7_38, U1.CN8_6
- new net N$5: LED1.A, R5.2
- new net N$6: DRIVER2.7
- new net ZEV: C3.1, C4.1, ENC-L.3, ENC-R.3, IC1.2, R1.2, R2.2, R3.2, R4.2
- net +3V3: no longer C3.1, C4.1, ENC-L.3, ENC-R.3, IC1.2, LCD.6, R1.2, R2.2, R3.2, R4.2
- net +7V: now also C5.1, C6.1, IC2.3
- net ENC_L_A: now also U1.CN10_29, U1.CN9_5; no longer U1.CN10_13, U1.CN5_5
- net ENC_L_B: now also U1.CN10_27, U1.CN9_6; no longer U1.CN10_15, U1.CN5_4
- net GND: now also C5.2, C6.2, C7.2, C8.2, IC2.1
- net LCD_BL: now also U1.CN10_23, U1.CN9_8
- net LCD_CE: now also U1.CN7_35
- net LCD_CLK: now also U1.CN10_11, U1.CN5_6
- net LCD_DC: now also U1.CN7_36, U1.CN8_5
- net LCD_DIN: now also U1.CN10_15, U1.CN5_4, U1.CN7_32, U1.CN8_3
- net LCD_RST: now also U1.CN7_37

Commit message: finished hardware & stm I2C problem
Parts:
- added C11: 100nF, rcl:C0402
- added S2: DTSM-3, dtsm3:DTSM-3
Connections:
- new net BUTTON1: C11.1, S2.2
- net GND_UC: now also U1.CN10_20, U1.CN10_9, U1.CN5_7
- net MOTOR_AIN_L: now also U1.CN10_24
- net MOTOR_AIN_R: now also U1.CN10_21, U1.CN5_1
- net MOTOR_BIN_L: now also U1.CN7_34, U1.CN8_4
- net MOTOR_BIN_R: now also U1.CN10_33, U1.CN9_3
- net N$1: now also C11.2, S2.1

Commit message: Adjusted wires.brd
Parts:
- removed C11: 100nF, rcl:C0402
- added C9: 100nF, capacitor-wima:C2.5-3
- moved S2 428.4 mm to (88.9, 92.7)
- moved LED1 409.7 mm to (143.5, 27.9), turned to 90 degrees
- moved R5 401.5 mm to (137.2, 30.5), turned to 270 degrees
- moved LCD 378.5 mm to (153.7, 29.2), turned to 90 degrees
- moved C8 349.7 mm to (31.8, 63.5), turned to 90 degrees
- moved C7 342.5 mm to (50.8, 38.1), turned to 90 degrees
- moved C6 342.4 mm to (53.3, 30.5), turned to 270 degrees
- moved DRIVER1 339.2 mm to (24.1, 85.1), turned to 180 degrees
- moved C5 334.1 mm to (36.8, 63.5), turned to 90 degrees
- moved DRIVER2 333.2 mm to (25.4, 71.1), turned to 180 degrees
- moved IC2 317.0 mm to (38.1, 30.5), turned to 90 degrees
- moved GYRO 316.4 mm to (99.1, 7.62), turned to 180 degrees
- moved VL-R 310.0 mm to (24.1, 92.7), turned to 180 degrees
- moved R4 304.5 mm to (58.4, 30.5), turned to 90 degrees
- moved C4 287.5 mm to (53.3, 57.1), turned to 90 degrees
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Connections:
- removed net GYRO_CS: GYRO.3
- removed net N$2: U1.CN7_38, U1.CN8_6
- removed net N$4: GYRO.10, GYRO.4
- net BUTTON1: now also C9.1, U1.CN10_4; no longer C11.1
- net ENC_L_A: now also U1.CN10_27, U1.CN9_6; no longer U1.CN10_29, U1.CN9_5
- net ENC_L_B: now also U1.CN10_29, U1.CN9_5; no longer U1.CN10_27, U1.CN9_6
- net GYRO_DEN: now also U1.CN10_14
- net GYRO_INT1: now also U1.CN10_12
- net GYRO_SCL: now also U1.CN10_17, U1.CN5_3
- net GYRO_SDA: now also U1.CN7_21
- net N$1: now also C9.2; no longer C11.2
- net VL_INT2: now also U1.CN10_34; no longer U1.CN10_16
- net ZEV: now also GYRO.10, GYRO.3, GYRO.4
Other:
- board size 160 x 100 mm -> 255.2 x 138.1 mm

Commit message: Board finished
Parts:
- moved C9 156.5 mm to (85.1, 91.4)
- moved LCD 71.0 mm to (121.9, 92.7), turned to 180 degrees
- moved POWER 46.7 mm to (62.2, 11.4), turned to 0 degrees
- moved R3 38.2 mm to (55.9, 31.8), turned to 90 degrees
- moved R5 34.9 mm to (108.0, 11.4), turned to 0 degrees
- moved R2 23.3 mm to (25.4, 52.1), turned to 0 degrees
- moved LED1 20.1 mm to (137.2, 8.89)
- moved R1 18.1 mm to (34.3, 20.3), turned to 0 degrees
- moved C1 14.2 mm to (39.4, 44.5)
- moved C4 14.2 mm to (39.4, 54.6)
- moved IC1 14.2 mm to (24.1, 44.5)
- moved IC2 14.2 mm to (24.1, 27.9)
- moved C2 14.2 mm to (43.2, 44.5)
- moved C3 14.2 mm to (34.3, 54.6)
- moved C5 14.2 mm to (22.9, 61.0)
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Routing:
- net GND: track 0.00 -> 274.9 mm, vias 0 -> 2
- net N$1: track 0.00 -> 138.1 mm
- net +3V3: track 0.00 -> 133.1 mm
- net GYRO_SCL: track 0.00 -> 112.1 mm
- net ZEV: track 0.00 -> 109.6 mm
- net GYRO_SDA: track 0.00 -> 70.4 mm
- net LS: track 0.00 -> 66.9 mm, vias 0 -> 2
- net VL_SCL: track 0.00 -> 62.5 mm, vias 0 -> 2
- net VL_SDA: track 0.00 -> 51.5 mm, vias 0 -> 5
- net +7V: track 0.00 -> 32.8 mm, vias 0 -> 2
- net N$5: track 0.00 -> 32.6 mm
- net ENC_R_A: track 0.00 -> 28.8 mm, vias 0 -> 1
- net M2R: track 0.00 -> 24.7 mm, vias 0 -> 1
- net MOTOR_BIN_L: track 0.00 -> 22.4 mm, vias 0 -> 1
- net BT_LED: track 0.00 -> 20.7 mm
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Other:
- board size 255.2 x 138.1 mm -> 144.8 x 102.5 mm
