File: hardware/mysz.sch (EAGLE design)
At the start: 30 parts, among them IC1 LM1117T(H)-3.3, IC2 LM1117T(H)-3.3, U1 NUCLEO-L053R8

Commit message: Adjusted wires.sch
Parts:
- removed C11: 100nF, rcl:C-EUC0402
- added C9: 100nF, capacitor-wima:C2,5-3
Connections:
- removed net GYRO_CS: GYRO.3
- removed net N$2: U1CN7.PC0_PB8/A5
- removed net N$4: GYRO.10, GYRO.4
- net BUTTON1: now also C9.1, U1CN10.PC6; no longer C11.1
- net ENC_L_A: now also U1CN10.PB4/D5; no longer U1CN10.PB5/D4
- net ENC_L_B: now also U1CN10.PB5/D4; no longer U1CN10.PB4/D5
- net GYRO_DEN: now also U1CN10.PA11
- net GYRO_INT1: now also U1CN10.PA12
- net GYRO_SCL: now also U1CN10.PB6/D10
- net GYRO_SDA: now also U1CN7.PB7
- net N$1: now also C9.2; no longer C11.2
- net VL_INT2: now also U1CN10.PC4; no longer U1CN10.PB12
- net ZEV: now also GYRO.10, GYRO.3, GYRO.4
Other:
- moved on the sheet: R3, R4
